Commit message: add relative path

File: arbot_model_pkg/urdf/ARbot_v2.urdf (robot description, URDF)
Before this commit: robot visual, 45 links, 44 joints
Links:
- link base_link: geometry visual mesh filename=package://arbot_model_pkg/meshes/STL/taz.stl scale=0.001 0.001 0.001
- link bedro_l: geometry visual mesh filename=package://arbot_model_pkg/meshes/STL/bedro.stl scale=0.001 0.001 0.001
- link bedro_r: geometry visual mesh filename=package://arbot_model_pkg/meshes/STL/bedro.stl scale=0.001 0.001 0.001
- link golen_l: geometry visual mesh filename=package://arbot_model_pkg/meshes/STL/golen.stl scale=0.001 0.001 0.001
- link golen_r: geometry visual mesh filename=package://arbot_model_pkg/meshes/STL/golen.stl scale=0.001 0.001 0.001
- link golova: geometry visual mesh filename=package://arbot_model_pkg/meshes/STL/golova.stl scale=0.001 0.001 0.001
- link golova_n: geometry visual mesh filename=package://arbot_model_pkg/meshes/STL/golovan.stl scale=0.001 0.001 0.001
- link kist_l: geometry visual mesh filename=package://arbot_model_pkg/meshes/STL/kist.stl scale=0.001 0.001 0.001
- link kist_r: geometry visual mesh filename=package://arbot_model_pkg/meshes/STL/kist.stl scale=0.001 0.001 0.001
- link koleno_l: geometry visual mesh filename=package://arbot_model_pkg/meshes/STL/koleno.stl scale=0.001 0.001 0.001
- link koleno_r: geometry visual mesh filename=package://arbot_model_pkg/meshes/STL/koleno.stl scale=0.001 0.001 0.001
- link kr_bedro_l: geometry visual mesh filename=package://arbot_model_pkg/meshes/STL/model2.stl scale=0.001 0.001 0.001
- link kr_bedro_r: geometry visual mesh filename=package://arbot_model_pkg/meshes/STL/model2.stl scale=0.001 0.001 0.001
- link kr_golova: geometry visual mesh filename=package://arbot_model_pkg/meshes/STL/model2.stl scale=0.001 0.001 0.001
- link kr_stopa_l: geometry visual mesh filename=package://arbot_model_pkg/meshes/STL/model2.stl scale=0.001 0.001 0.001
- link kr_stopa_r: geometry visual mesh filename=package://arbot_model_pkg/meshes/STL/model2.stl scale=0.001 0.001 0.001
- link lokot_l: geometry visual mesh filename=package://arbot_model_pkg/meshes/STL/model13.stl scale=0.001 0.001 0.001
- link lokot_r: geometry visual mesh filename=package://arbot_model_pkg/meshes/STL/model13.stl scale=0.001 0.001 0.001
- link plecho_l: geometry visual mesh filename=package://arbot_model_pkg/meshes/STL/model10.stl scale=0.001 0.001 0.001
- link plecho_r: geometry visual mesh filename=package://arbot_model_pkg/meshes/STL/model10.stl scale=0.001 0.001 0.001
- link predpl_l: geometry visual mesh filename=package://arbot_model_pkg/meshes/STL/model13.stl scale=0.001 0.001 0.001
- link predpl_r: geometry visual mesh filename=package://arbot_model_pkg/meshes/STL/model13.stl scale=0.001 0.001 0.001
- link sh_bedro1_l: geometry visual mesh filename=package://arbot_model_pkg/meshes/STL/model6.stl scale=0.001 0.001 0.001
- link sh_bedro1_r: geometry visual mesh filename=package://arbot_model_pkg/meshes/STL/model6.stl scale=0.001 0.001 0.001
- link sh_bedro_l: geometry visual mesh filename=package://arbot_model_pkg/meshes/STL/model7.stl scale=0.001 0.001 0.001
- link sh_bedro_r: geometry visual mesh filename=package://arbot_model_pkg/meshes/STL/model7.stl scale=0.001 0.001 0.001
- link sh_golova_n: geometry visual mesh filename=package://arbot_model_pkg/meshes/STL/koleno.stl scale=0.001 0.001 0.001
- link sh_kist_l: geometry visual mesh filename=package://arbot_model_pkg/meshes/STL/model7.stl scale=0.001 0.001 0.001
- link sh_kist_r: geometry visual mesh filename=package://arbot_model_pkg/meshes/STL/model7.stl scale=0.001 0.001 0.001
- link sh_lokot1_l: geometry visual mesh filename=package://arbot_model_pkg/meshes/STL/model6.stl scale=0.001 0.001 0.001
- link sh_lokot1_r: geometry visual mesh filename=package://arbot_model_pkg/meshes/STL/model6.stl scale=0.001 0.001 0.001
- link sh_lokot_l: geometry visual mesh filename=package://arbot_model_pkg/meshes/STL/model7.stl scale=0.001 0.001 0.001
- link sh_lokot_r: geometry visual mesh filename=package://arbot_model_pkg/meshes/STL/model7.stl scale=0.001 0.001 0.001
- link sh_plecho1_l: geometry visual mesh filename=package://arbot_model_pkg/meshes/STL/koleno.stl scale=0.001 0.001 0.001
- link sh_plecho1_r: geometry visual mesh filename=package://arbot_model_pkg/meshes/STL/koleno.stl scale=0.001 0.001 0.001
- link sh_plecho_l: geometry visual mesh filename=package://arbot_model_pkg/meshes/STL/model11.stl scale=0.001 0.001 0.001
- link sh_plecho_r: geometry visual mesh filename=package://arbot_model_pkg/meshes/STL/model11.stl scale=0.001 0.001 0.001
- link sh_predpl_l: geometry visual mesh filename=package://arbot_model_pkg/meshes/STL/koleno.stl scale=0.001 0.001 0.001
- link sh_predpl_r: geometry visual mesh filename=package://arbot_model_pkg/meshes/STL/koleno.stl scale=0.001 0.001 0.001
- link sh_sheya: geometry visual mesh filename=package://arbot_model_pkg/meshes/STL/sheya.stl scale=0.001 0.001 0.001
- link sh_tors: geometry visual mesh filename=package://arbot_model_pkg/meshes/STL/model7.stl scale=0.001 0.001 0.001
- link sheya: geometry visual mesh filename=package://arbot_model_pkg/meshes/STL/model10.stl scale=0.001 0.001 0.001
- link stopa_l: geometry visual mesh filename=package://arbot_model_pkg/meshes/STL/stopa.stl scale=0.001 0.001 0.001
- link stopa_r: geometry visual mesh filename=package://arbot_model_pkg/meshes/STL/stopa.stl scale=0.001 0.001 0.001
- link tors: geometry visual mesh filename=package://arbot_model_pkg/meshes/STL/tors.stl scale=0.001 0.001 0.001
